File: hardware/pcb/QuadPower/Current/powerattempt9wout.sch (EAGLE design)
At the start: 74 parts, among them IC1 24LC128ST, IC2 INA168, IC3 INA168, IC4 INA168, IC5 INA168, IC6 INA168, IC7 INA168, IC8 INA168, IC9 INA168

Commit message: Added REV-A and the current QuadPower Boards, removed old files
Parts:
- added 3V3INDUC, 5VINDUC, SPOWINDUC: 1200RS, inductors:1200RS
- added C17, C18, C19, C20, C21, C22, C23, C24, C25: 10uF, SparkFun:CAP1206
- added C27: 100uF, SparkFun:CAP1206
- added D1, D2, D3: (no value), diode:SCHOTTKY-DIODESMD
- added JP10, JP11, JP12, JP13, JP14, JP15, JP16, JP17, JP18, JP19, JP2, JP20, JP21, JP22, JP23, JP24, JP25, JP3, JP4, JP5, JP6, JP7, JP8, JP9: (no value), SparkFun:M03PTH
- added JP26, JP27: (no value), SparkFun:M06SIP
- added LED1, LED2, LED3, LED4, LED5: (no value), led:LEDSML0805
- added R42, R43, R46, R50, R51: (no value), SparkFun:RESISTOR0805-RES
- added R44, R47, R48: 1.69k 1%, SparkFun:RESISTOR0805-RES
- added R45: 4.7k 0.1%, SparkFun:RESISTOR0805-RES
- added R49: (no value), resistor:R-US_M0805
- added SV1, SV2: (no value), con-lstb:MA08-1
- added SV25: (no value), con-lstb:MA04-1
- added SV26: (no value), con-lstb:MA07-1
- added SV27: (no value), con-lstb:MA06-1
- added SW1, SW2: SWS008, smd-special:SWS008
- added U$10: Motor3, SparkFun:DEANSDEANS
- added U$11: Motor4, SparkFun:DEANSDEANS
- added U$12: Logic, SparkFun:DEANSDEANS
- added U$4, U$5, U$6: AP1509, SparkFun:AP1509
- added U$7: INPUT, SparkFun:DEANSDEANS
- added U$8: Motor1, SparkFun:DEANSDEANS
- added U$9: Motor2, SparkFun:DEANSDEANS
- R11, R16, R21, R26, R31, R36, R41, R6: device rcl:R-US_R2512 -> SparkFun:LVK25
Connections:
- removed net 3V3: U$2.VCCA, U$3.VCCA
- removed net DOUT: X1.DOUT, X2.DOUT, X3.DOUT
- removed net N$10: IC3.IN-, R11.2, R7.1
- removed net N$11: IC3.IN+, IC3.V+, R11.1
- removed net N$14: IC4.IN-, R12.1, R16.2
- removed net N$15: IC4.IN+, IC4.V+, R16.1
- removed net N$17: IC5.IN-, R17.1, R21.2
- removed net N$18: IC5.IN+, IC5.V+, R21.1
- removed net N$20: IC6.IN-, R22.1, R26.2
- removed net N$21: IC6.IN+, IC6.V+, R26.1
- removed net N$23: IC7.IN-, R27.1, R31.2
- removed net N$24: IC7.IN+, IC7.V+, R31.1
- removed net N$26: IC8.IN-, R32.1, R36.2
- removed net N$27: IC8.IN+, IC8.V+, R36.1
- removed net N$29: IC9.IN-, R37.1, R41.2
- removed net N$30: IC9.IN+, IC9.V+, R41.1
- removed net N$8: IC2.IN-, R2.1, R6.2
- removed net N$9: IC2.IN+, IC2.V+, R6.1
- new net 3V3CUR: 3V3INDUC.2, C23.1, IC6.IN+, IC6.V+, R22.1, R26.1, R45.2
- new net 5VCUR: 5VINDUC.2, C22.1, IC8.IN+, IC8.V+, R32.1, R36.1, U$5.FB
- new net A0: JP5.1, X3.CH0
- new net A1: JP4.1, X3.CH1
- new net A2: JP3.1, X3.CH2
- new net A3: JP2.1, X3.CH3
- new net A4: JP9.1, X3.CH4
- new net A5: JP8.1, X3.CH5
- new net A6: JP7.1, X3.CH6
- new net A7: JP6.1, X3.CH7
- new net EC0: SV2.8, SW2.9, U$1P8X32A-Q44.P12
- new net EC1: SV2.7, SW2.10, U$1P8X32A-Q44.P11
- new net EC2: SV2.6, SW2.11, U$1P8X32A-Q44.P10
- new net EC3: SV2.5, SW2.12, U$1P8X32A-Q44.P9
- new net ECSP0: JP18.2
- new net ECSP1: JP19.2
- new net ECSP2: JP20.2
- new net ECSP3: JP21.2
- new net IMU_RX: SV25.3, U$1P8X32A-Q44.P27
- new net IMU_TX: SV25.4, U$1P8X32A-Q44.P26
- new net LOGICBAT: IC4.IN+, IC4.V+, R12.1, R16.1, U$12.1
- new net LOGICPOW: IC4.IN-, R16.2, U$4.VIN, U$5.VIN
- new net M1: IC9.IN+, IC9.V+, R37.1, R41.1, U$8.1
- new net M2: IC7.IN+, IC7.V+, R27.1, R31.1, U$9.1
- new net M3: IC5.IN+, IC5.V+, R17.1, R21.1, U$10.1
- new net M4: IC3.IN+, IC3.V+, R11.1, R7.1, U$11.1
- new net MOTORBAT: IC3.IN-, IC5.IN-, IC7.IN-, IC9.IN-, R11.2, R21.2, R31.2, R41.2, U$6.VIN, U$7.1
- new net N$71: LED1.C, R46.2
- new net N$72: LED2.C, R43.2
- new net N$73: LED3.C, R42.2
- new net N$77: 3V3INDUC.1, D2.C, U$4.VOUT
- new net N$78: 5VINDUC.1, D1.C, U$5.VOUT
- new net N$79: D3.C, SPOWINDUC.1, U$6.VOUT
- new net N$83: R44.1, R45.1, U$4.FB
- new net N0: LED5.A, SV2.4, SW2.13, U$1P8X32A-Q44.P8
- new net N1: LED4.A, SV2.3, SW2.14, U$1P8X32A-Q44.P7
- new net N2: SV2.2, SW2.15, U$1P8X32A-Q44.P6
- new net N3: SV2.1, SW2.16, U$1P8X32A-Q44.P5
- new net S0: SV1.8, SW1.9, U$1P8X32A-Q44.P20
- new net S1: SV1.7, SW1.10, U$1P8X32A-Q44.P19
- new net S2: SV1.6, SW1.11, U$1P8X32A-Q44.P18
- new net S3: SV1.5, SW1.12, U$1P8X32A-Q44.P17
- new net S4: SV1.4, SW1.13, U$1P8X32A-Q44.P16
- new net S5: SV1.3, SW1.14, U$1P8X32A-Q44.P15
- new net S6: SV1.2, SW1.15, U$1P8X32A-Q44.P14
- new net S7: SV1.1, SW1.16, U$1P8X32A-Q44.P13
- new net SCL: IC1.SCL, R49.2, SV27.3, U$1P8X32A-Q44.P28
- new net SD0: SV26.3, U$1P8X32A-Q44.P0
- new net SD1: SV26.4, U$1P8X32A-Q44.P1
- new net SD2: SV26.5, U$1P8X32A-Q44.P2
- new net SD3: SV26.6, U$1P8X32A-Q44.P3
- new net SD4: SV26.7, U$1P8X32A-Q44.P4
- new net SDA: IC1.SDA, R1.1, SV27.2, U$1P8X32A-Q44.P29
- new net SPOW: IC2.IN-, JP10.2, JP11.2, JP12.2, JP13.2, JP14.2, JP15.2, JP16.2, JP17.2, LED1.A, R6.2
- new net SPOWCUR: C21.1, IC2.IN+, IC2.V+, R2.1, R6.1, SPOWINDUC.2, U$6.FB
- net 5V: now also C18.2, C19.2, C20.2, IC8.IN-, JP2.2, JP22.2, JP23.2, JP24.2, JP25.2, JP26.1, JP26.4, JP27.1, JP27.4, JP3.2, JP4.2, JP5.2, JP6.2, JP7.2, JP8.2, JP9.2, LED3.A, R36.2, SV25.1, SV27.6, X1.VDD, X1.VREF, X2.VDD, X2.VREF, X3.VDD, X3.VREF
- net BREAKOUT_0: now also JP22.1
- net BREAKOUT_1: now also JP23.1
- net BREAKOUT_2: now also JP24.1
- net BREAKOUT_3: now also JP25.1
- net CLK: now also U$1P8X32A-Q44.P25
- net CS1: now also U$1P8X32A-Q44.P23
- net CS2: now also U$1P8X32A-Q44.P22
- net CS3: now also U$1P8X32A-Q44.P21
- net DIN: now also U$1P8X32A-Q44.P24, X1.DOUT, X2.DOUT, X3.DOUT
- net ECS0: now also JP18.1
- net ECS1: now also JP19.1
- net ECS2: now also JP20.1
- net ECS3: now also JP21.1
- net GND: now also C17.2, C18.1, C19.1, C20.1, C21.2, C22.2, C23.2, C24.2, C25.2, C27.1, D1.A, D2.A, D3.A, JP10.3, JP11.3, JP12.3, JP13.3, JP14.3, JP15.3, JP16.3, JP17.3, JP18.3, JP19.3, JP2.3, JP20.3, JP21.3, JP22.3, JP23.3, JP24.3, JP25.3, JP26.2, JP26.5, JP27.2, JP27.5, JP3.3, JP4.3, JP5.3, JP6.3, JP7.3, JP8.3, JP9.3, R42.1, R43.1, R44.2, R46.1, R50.1, R51.1, SV25.2, SV26.2, SV27.1, SV27.5, U$10.2, U$11.2, U$12.2, U$1P8X32A-Q44.BOE/, U$4.GND, U$4.SD, U$5.GND, U$5.SD, U$6.GND, U$6.SD, U$7.2, U$8.2, U$9.2, X1.AGND, X1.DGND, X2.AGND, X2.DGND, X3.AGND, X3.DGND
- net N$1: now also R47.2
- net N$2: now also R48.2
- net N$3: now also LED4.C, R50.2; no longer IC1.SCL, U$1P8X32A-Q44.P28
- net N$32: now also SW1.8
- net N$33: now also SW1.7
- net N$34: now also SW1.6
- net N$35: now also SW1.5
- net N$36: now also SW1.4
- net N$37: now also SW1.3
- net N$38: now also SW1.2
- net N$39: now also SW1.1
- net N$4: now also LED5.C, R51.2; no longer IC1.SDA, R1.1, U$1P8X32A-Q44.P29
- net N$41: now also SW2.8
- net N$42: now also SW2.7
- net N$43: now also SW2.6
- net N$44: now also SW2.5
- net N$45: now also SW2.4
- net N$46: now also SW2.3
- net N$47: now also SW2.2
- net N$48: now also SW2.1
- net SERVO_0: now also JP10.1
- net SERVO_1: now also JP11.1
- net SERVO_2: now also JP12.1
- net SERVO_3: now also JP13.1
- net SERVO_4: now also JP14.1
- net SERVO_5: now also JP15.1
- net SERVO_6: now also JP16.1
- net SERVO_7: now also JP17.1
- net VDD: now also C17.1, C24.1, C25.1, C27.2, IC6.IN-, JP26.3, JP26.6, JP27.3, JP27.6, LED2.A, R26.2, R47.1, R48.1, R49.1, SV26.1, SV27.4, U$2.VCCA, U$3.VCCA
Other:
- moved on the sheet: C1, C11, C13, C15, C3, C5, C7, C9, R12, R13, R14, R17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
